File: BME280.sch (KiCad schematic (older format))
At the start: 4 parts, among them J8 BME280_(GYBMEP), U4 BME280

Commit message: Add JCLPCB/LCSC part numbers
Parts:
- C11, C12: LCSC (none) -> C49678
Changed lines of the file:
@@
 EESchema Schematic File Version 4
+LIBS:ULPSoilMonitor-cache
 EELAYER 30 0
 EELAYER END
@@
 F 2 "Capacitor_SMD:C_0805_2012Metric" H 2238 1400 50  0001 C CNN
 F 3 "~" H 2200 1550 50  0001 C CNN
+F 4 "C49678" H 2200 1550 50  0001 C CNN "LCSC"
 	1    2200 1550
 	1    0    0    -1
@@
 F 2 "Capacitor_SMD:C_0805_2012Metric" H 1988 1700 50  0001 C CNN
 F 3 "~" H 1950 1850 50  0001 C CNN
+F 4 "C49678" H 1950 1850 50  0001 C CNN "LCSC"
 	1    1950 1850
 	1    0    0    -1
