File: SensorHeaders.sch (KiCad schematic (older format))
At the start: 22 parts, among them J1 Conn_01x03_Male, J2 Conn_01x03_Male, J3 Conn_01x03_Male, J4 Conn_01x03_Male, J5 Conn_01x03_Male, J6 Conn_01x03_Male, Q1 BC807

Commit message: Add JCLPCB/LCSC part numbers
Parts:
- Q1: LCSC (none) -> C8587
- R10, R11, R16, R17, R18, R8, R9: LCSC (none) -> C17621
- R12, R13, R14, R4, R5, R6, R7: LCSC (none) -> C17801
- R15: LCSC (none) -> C17614
Changed lines of the file:
@@
 EESchema Schematic File Version 4
+LIBS:ULPSoilMonitor-cache
 EELAYER 30 0
 EELAYER END
@@
 F 2 "Resistor_SMD:R_0805_2012Metric" V 1780 1250 50  0001 C CNN
 F 3 "~" H 1850 1250 50  0001 C CNN
+F 4 "C17801" H 1850 1250 50  0001 C CNN "LCSC"
 	1    1850 1250
 	1    0    0    -1
@@
 F 2 "Resistor_SMD:R_0805_2012Metric" V 1780 1750 50  0001 C CNN
 F 3 "~" H 1850 1750 50  0001 C CNN
+F 4 "C17621" H 1850 1750 50  0001 C CNN "LCSC"
 	1    1850 1750
 	1    0    0    -1
@@
 F 2 "Resistor_SMD:R_0805_2012Metric" V 2780 1250 50  0001 C CNN
 F 3 "~" H 2850 1250 50  0001 C CNN
+F 4 "C17801" H 2850 1250 50  0001 C CNN "LCSC"
 	1    2850 1250
 	1    0    0    -1
@@
 F 2 "Resistor_SMD:R_0805_2012Metric" V 2780 1750 50  0001 C CNN
 F 3 "~" H 2850 1750 50  0001 C CNN
+F 4 "C17621" H 2850 1750 50  0001 C CNN "LCSC"
 	1    2850 1750
 	1    0    0    -1
@@
 F 2 "Resistor_SMD:R_0805_2012Metric" V 3780 1250 50  0001 C CNN
 F 3 "~" H 3850 1250 50  0001 C CNN
+F 4 "C17801" H 3850 1250 50  0001 C CNN "LCSC"
 	1    3850 1250
 	1    0    0    -1
@@
 F 2 "Resistor_SMD:R_0805_2012Metric" V 3780 1750 50  0001 C CNN
 F 3 "~" H 3850 1750 50  0001 C CNN
+F 4 "C17621" H 3850 1750 50  0001 C CNN "LCSC"
 	1    3850 1750
 	1    0    0    -1
@@
 F 2 "Resistor_SMD:R_0805_2012Metric" V 1780 2600 50  0001 C CNN
 F 3 "~" H 1850 2600 50  0001 C CNN
+F 4 "C17801" H 1850 2600 50  0001 C CNN "LCSC"
 	1    1850 2600
 	1    0    0    -1
@@
 F 2 "Resistor_SMD:R_0805_2012Metric" V 1780 3100 50  0001 C CNN
 F 3 "~" H 1850 3100 50  0001 C CNN
+F 4 "C17621" H 1850 3100 50  0001 C CNN "LCSC"
 	1    1850 3100
 	1    0    0    -1
@@
 F 2 "Resistor_SMD:R_0805_2012Metric" V 2780 2600 50  0001 C CNN
 F 3 "~" H 2850 2600 50  0001 C CNN
+F 4 "C17801" H 2850 2600 50  0001 C CNN "LCSC"
 	1    2850 2600
 	1    0    0    -1
@@
 F 2 "Resistor_SMD:R_0805_2012Metric" V 2780 3100 50  0001 C CNN
 F 3 "~" H 2850 3100 50  0001 C CNN
+F 4 "C17621" H 2850 3100 50  0001 C CNN "LCSC"
 	1    2850 3100
 	1    0    0    -1
@@
 F 2 "Resistor_SMD:R_0805_2012Metric" V 3780 2600 50  0001 C CNN
 F 3 "~" H 3850 2600 50  0001 C CNN
+F 4 "C17801" H 3850 2600 50  0001 C CNN "LCSC"
 	1    3850 2600
 	1    0    0    -1
@@
 F 2 "Resistor_SMD:R_0805_2012Metric" V 3780 3100 50  0001 C CNN
 F 3 "~" H 3850 3100 50  0001 C CNN
+F 4 "C17621" H 3850 3100 50  0001 C CNN "LCSC"
 	1    3850 3100
 	1    0    0    -1
@@
 F 2 "Resistor_SMD:R_0805_2012Metric" V 9230 1250 50  0001 C CNN
 F 3 "~" H 9300 1250 50  0001 C CNN
+F 4 "C17801" H 9300 1250 50  0001 C CNN "LCSC"
 	1    9300 1250
 	1    0    0    -1
@@
 F 2 "Resistor_SMD:R_0805_2012Metric" V 9230 1750 50  0001 C CNN
 F 3 "~" H 9300 1750 50  0001 C CNN
+F 4 "C17621" H 9300 1750 50  0001 C CNN "LCSC"
 	1    9300 1750
 	1    0    0    -1
@@
 F 2 "Package_TO_SOT_SMD:SOT-23" H 9100 2575 50  0001 L CIN
 F 3 "http://www.fairchildsemi.com/ds/BC/BC807.pdf" H 8900 2650 50  0001 L CNN
+F 4 "C8587" H 8900 2650 50  0001 C CNN "LCSC"
 	1    8900 2650
 	-1   0    0    1
@@
 F 2 "Resistor_SMD:R_0805_2012Metric" V 9280 2650 50  0001 C CNN
 F 3 "~" H 9350 2650 50  0001 C CNN
+F 4 "C17614" H 9350 2650 50  0001 C CNN "LCSC"
 	1    9350 2650
 	0    1    1    0
